Commit message: 增加机械臂，且能导航

File: Week-7-8-ROS2-Navigation/bme_ros2_navigation/urdf/macros.xacro (robot description, xacro)
@@ -291,4 +291,35 @@
       </visual>
     </link>
+    <!-- Arm Mount Link for MyCobot -->
+    <link name="${link_prefix}mycobot_arm_mount_link">
+      <inertial>
+        <mass value="0.01"/>
+        <origin xyz="0 0 0" rpy="0 0 0"/>
+        <inertia
+            ixx="1e-6" ixy="0" ixz="0"
+            iyy="1e-6" iyz="0"
+            izz="1e-6"
+        />
+      </inertial>
+      <visual>
+        <origin xyz="0 0 0" rpy="0 0 0"/>
+        <geometry>
+          <box size="0.01 0.01 0.01"/>
+        </geometry>
+      </visual>
+    </link>
+    <joint name="${joint_prefix}arm_mount_joint" type="fixed">
+      <origin xyz="0.0 0.0 0.15" rpy="0 0 0"/>
+      <parent link="${link_prefix}base_link"/>
+      <child link="${link_prefix}mycobot_arm_mount_link"/>
+    </joint>
+    <!-- Include MyCobot Arm -->
+    <xacro:include filename="$(find bme_ros2_navigation)/urdf/mycobot/mycobot_280_arm.urdf.xacro"/>
+    <xacro:mycobot_280_arm
+      base_link="arm_mount_link"
+      flange_link="link6_flange"
+      prefix="${link_prefix}mycobot_">
+      <origin xyz="0 0 0" rpy="0 0 0"/>
+    </xacro:mycobot_280_arm>
   </xacro:macro>
   <!-- LEO GAZEBO -->

Commit message: 机械臂移到前面，雷达在中间且不悬浮。问题：map jump严重，或许可稍微抬高雷达

File: Week-7-8-ROS2-Navigation/bme_ros2_navigation/urdf/macros.xacro (robot description, xacro)
@@ -264,5 +264,5 @@
     <!-- Lidar -->
     <joint name="${joint_prefix}scan_joint" type="fixed">
-      <origin xyz="0.0 0 0.15" rpy="0 0 0"/>
+      <origin xyz="0.0 0 0.0" rpy="0 0 0"/>
       <child link="${link_prefix}scan_link"/>
       <parent link="${link_prefix}base_link"/>
@@ -270,10 +270,10 @@
     <link name="${link_prefix}scan_link">
       <inertial>
-        <mass value="1e-5"/>
+        <mass value="0.19"/>
         <origin xyz="0 0 0" rpy="0 0 0"/>
         <inertia
-            ixx="1e-6" ixy="0" ixz="0"
-            iyy="1e-6" iyz="0"
-            izz="1e-6"
+            ixx="0.0001" ixy="0" ixz="0"
+            iyy="0.0001" iyz="0"
+            izz="0.0001"
         />
       </inertial>
@@ -281,5 +281,5 @@
         <origin xyz="0 0 0" rpy="0 0 0"/>
         <geometry>
-          <box size=".1 .1 .1"/>
+          <cylinder radius="0.038" length="0.041"/>
         </geometry>
       </collision>
@@ -287,5 +287,5 @@
         <origin xyz="0 0 0" rpy="0 0 0"/>
         <geometry>
-          <cylinder radius="0.05" length="0.1"/>
+          <cylinder radius="0.038" length="0.041"/>
         </geometry>
       </visual>
@@ -310,5 +310,5 @@
     </link>
     <joint name="${joint_prefix}arm_mount_joint" type="fixed">
-      <origin xyz="0.0 0.0 0.15" rpy="0 0 0"/>
+      <origin xyz="0.08 0.0 0.0" rpy="0 0 0"/>
       <parent link="${link_prefix}base_link"/>
       <child link="${link_prefix}mycobot_arm_mount_link"/>
@@ -556,5 +556,5 @@
           </scan>
           <range>
-            <min>0.05</min>
+            <min>0.25</min>
             <max>10.0</max>
             <resolution>0.01</resolution>

Commit message: 雷达放在中间，机械臂抬高6cm并给一个力让他不垂

File: Week-7-8-ROS2-Navigation/bme_ros2_navigation/urdf/macros.xacro (robot description, xacro)
@@ -310,5 +310,5 @@
     </link>
     <joint name="${joint_prefix}arm_mount_joint" type="fixed">
-      <origin xyz="0.08 0.0 0.0" rpy="0 0 0"/>
+      <origin xyz="0.08 0.0 0.06" rpy="0 0 0"/>
       <parent link="${link_prefix}base_link"/>
       <child link="${link_prefix}mycobot_arm_mount_link"/>

File: Week-7-8-ROS2-Navigation/bme_ros2_navigation/urdf/mycobot/mycobot_280_arm.urdf.xacro (robot description, xacro)
@@ -199,4 +199,64 @@
     <xacro:material_visual ref_link="${prefix}link6" ambient="1 1 1 1" diffuse="1 1 1 1" specular="1 1 1 1"/>
     <xacro:material_visual ref_link="${prefix}${flange_link}" ambient="0.5 0.5 0.5 1" diffuse="0.5 0.5 0.5 1" specular="0.5 0.5 0.5 1"/>
+    <!-- ros2_control configuration -->
+    <ros2_control name="${prefix}mycobot_arm" type="system">
+      <hardware>
+        <plugin>gz_ros2_control/GazeboSimSystem</plugin>
+      </hardware>
+      <joint name="${prefix}link1_to_${prefix}link2">
+        <command_interface name="position">
+          <param name="min">-2.879793</param>
+          <param name="max">2.879793</param>
+        </command_interface>
+        <state_interface name="position"/>
+        <state_interface name="velocity"/>
+      </joint>
+      <joint name="${prefix}link2_to_${prefix}link3">
+        <command_interface name="position">
+          <param name="min">-2.879793</param>
+          <param name="max">2.879793</param>
+        </command_interface>
+        <state_interface name="position"/>
+        <state_interface name="velocity"/>
+      </joint>
+      <joint name="${prefix}link3_to_${prefix}link4">
+        <command_interface name="position">
+          <param name="min">-2.879793</param>
+          <param name="max">2.879793</param>
+        </command_interface>
+        <state_interface name="position"/>
+        <state_interface name="velocity"/>
+      </joint>
+      <joint name="${prefix}link4_to_${prefix}link5">
+        <command_interface name="position">
+          <param name="min">-2.879793</param>
+          <param name="max">2.879793</param>
+        </command_interface>
+        <state_interface name="position"/>
+        <state_interface name="velocity"/>
+      </joint>
+      <joint name="${prefix}link5_to_${prefix}link6">
+        <command_interface name="position">
+          <param name="min">-2.879793</param>
+          <param name="max">2.879793</param>
+        </command_interface>
+        <state_interface name="position"/>
+        <state_interface name="velocity"/>
+      </joint>
+      <joint name="${prefix}link6_to_${prefix}${flange_link}">
+        <command_interface name="position">
+          <param name="min">-3.05</param>
+          <param name="max">3.05</param>
+        </command_interface>
+        <state_interface name="position"/>
+        <state_interface name="velocity"/>
+      </joint>
+    </ros2_control>
+    <!-- Gazebo ros2_control plugin -->
+    <gazebo>
+      <plugin filename="gz_ros2_control-system" name="gz_ros2_control::GazeboSimROS2ControlPlugin">
+        <parameters>$(find bme_ros2_navigation)/config/mycobot_controllers.yaml</parameters>
+      </plugin>
+    </gazebo>
   </xacro:macro>
 </robot>

Commit message: 1.解决机械臂装在车头导致重心前移，小车轻微'点头'（前倾），使水平安装的雷达扫到了远处的地面。2.地图刷新频率：从 5.0秒 提升到 1.0秒 (快了5倍) 3.扫描处理速度：从 0.5秒 提升到 0.2秒 4.容错时间：增加到 0.5秒，防止因卡顿导致的数据丢失

File: Week-7-8-ROS2-Navigation/bme_ros2_navigation/urdf/macros.xacro (robot description, xacro)
@@ -264,5 +264,5 @@
     <!-- Lidar -->
     <joint name="${joint_prefix}scan_joint" type="fixed">
-      <origin xyz="0.0 0 0.0" rpy="0 0 0"/>
+      <origin xyz="0.0 0 0.02" rpy="0 -0.035 0"/>
       <child link="${link_prefix}scan_link"/>
       <parent link="${link_prefix}base_link"/>
@@ -556,5 +556,5 @@
           </scan>
           <range>
-            <min>0.25</min>
+            <min>0.10</min>
             <max>10.0</max>
             <resolution>0.01</resolution>

Commit message: 增加机械臂moveit抓取仿真功能，实现根据坐标向下抓取（无视了机身），而且该版本下导航仿真非常流畅

File: Week-7-8-ROS2-Navigation/bme_ros2_navigation/urdf/macros.xacro (robot description, xacro)
@@ -322,4 +322,11 @@
       <origin xyz="0 0 0" rpy="0 0 0"/>
     </xacro:mycobot_280_arm>
+    <!-- Include Adaptive Gripper -->
+    <xacro:include filename="$(find mycobot_description)/urdf/mech/adaptive_gripper.urdf.xacro"/>
+    <xacro:adaptive_gripper
+      parent="link6_flange"
+      prefix="${link_prefix}mycobot_">
+      <origin xyz="0 0 0.034" rpy="1.5708 0 0"/>
+    </xacro:adaptive_gripper>
   </xacro:macro>
   <!-- LEO GAZEBO -->

File: Week-7-8-ROS2-Navigation/bme_ros2_navigation/urdf/mycobot/mycobot_280_arm.urdf.xacro (robot description, xacro)
@@ -252,4 +252,13 @@
         <state_interface name="velocity"/>
       </joint>
+      <!-- Gripper controller joint -->
+      <joint name="${prefix}gripper_controller">
+        <command_interface name="position">
+          <param name="min">-0.7</param>
+          <param name="max">0.15</param>
+        </command_interface>
+        <state_interface name="position"/>
+        <state_interface name="velocity"/>
+      </joint>
     </ros2_control>
     <!-- Gazebo ros2_control plugin -->
