Commit message: 修改机械臂底座，将其和真的安装方向设置一致

File: Week-7-8-ROS2-Navigation/bme_ros2_navigation/urdf/mycobot/mycobot_280_arm.urdf.xacro (robot description, xacro)
@@ -40,5 +40,5 @@
           <mesh filename="package://bme_ros2_navigation/meshes/mycobot_280/visual/link1.dae"/>
         </geometry>
-        <origin xyz="0.0 0 0" rpy="0 0 ${-pi/2}"/>
+        <origin xyz="0.0 0 0" rpy="0 0 ${-pi}"/>
       </visual>
       <collision>
